File: Stepperansteuerung/StepperControl.sch (KiCad schematic (older format))
At the start: 2 parts

Commit message: Steppercontrol Update
Parts:
- added U?: Stepper, symbol Stepper
Connections:
- net at U?.11 (1B): now also U?.4 (1B)
- net at U?.12 (1A): now also U?.3 (1A)
- net at U?.13 (2A): now also U?.2 (2A)
- net at U?.14 (2B): now also U?.1 (2B)
Changed lines of the file:
@@
 LIBS:tcxo
 LIBS:polulu
+LIBS:StepperControl-cache
 EELAYER 25 0
 EELAYER END
@@
 Wire Wire Line
 	6550 3400 6250 3400
+$Comp
+L Stepper U?
+U 1 1 58B01121
+P 7300 3650
+F 0 "U?" H 7050 4000 60  0000 C CNN
+F 1 "Stepper" H 7150 3300 60  0000 C CNN
+F 2 "" H 7300 3650 60  0000 C CNN
+F 3 "" H 7300 3650 60  0000 C CNN
+	1    7300 3650
+	1    0    0    -1
+$EndComp
+Wire Wire Line
+	6250 3500 6800 3500
+Wire Wire Line
+	6250 3600 6800 3600
+Wire Wire Line
+	6250 3700 6800 3700
+Wire Wire Line
+	6250 3800 6800 3800
 $EndSCHEMATC
