File: Stepperansteuerung/StepperControl.sch (KiCad schematic (older format))
At the start: 3 parts

Commit message: Update Stepperansteuerung
Parts:
- added P? (x2): CONN_01X04, symbol CONN_01X04
Connections:
- wire segments 18 -> 22
Other:
- moved on the sheet: U?
Changed lines of the file:
@@
 LIBS:linear_tech
 LIBS:micrel
-LIBS:microchip_power
 LIBS:NDK
 LIBS:newhaven
@@
 L Stepper U?
 U 1 1 58B01121
-P 8200 3650
-F 0 "U?" H 7950 4000 60  0000 C CNN
-F 1 "Stepper" H 8050 3300 60  0000 C CNN
-F 2 "" H 8200 3650 60  0000 C CNN
-F 3 "" H 8200 3650 60  0000 C CNN
-	1    8200 3650
+P 9600 3650
+F 0 "U?" H 9350 4000 60  0000 C CNN
+F 1 "Stepper" H 9450 3300 60  0000 C CNN
+F 2 "" H 9600 3650 60  0000 C CNN
+F 3 "" H 9600 3650 60  0000 C CNN
+	1    9600 3650
 	1    0    0    -1
 $EndComp
 Wire Wire Line
-	6250 3500 6800 3500
+	6250 3500 7100 3500
 Wire Wire Line
-	6250 3600 6800 3600
+	6250 3600 7100 3600
 Wire Wire Line
-	6250 3700 6800 3700
+	6250 3700 7100 3700
 Wire Wire Line
-	6250 3800 6800 3800
+	6250 3800 7100 3800
+$Comp
+L CONN_01X04 P?
+U 1 1 58D04B64
+P 7300 3650
+F 0 "P?" H 7300 3900 50  0000 C CNN
+F 1 "CONN_01X04" V 7400 3650 50  0000 C CNN
+F 2 "" H 7300 3650 50  0000 C CNN
+F 3 "" H 7300 3650 50  0000 C CNN
+	1    7300 3650
+	1    0    0    -1
+$EndComp
+$Comp
+L CONN_01X04 P?
+U 1 1 58D04BB1
+P 8100 3650
+F 0 "P?" H 8100 3900 50  0000 C CNN
+F 1 "CONN_01X04" V 8200 3650 50  0000 C CNN
+F 2 "" H 8100 3650 50  0000 C CNN
+F 3 "" H 8100 3650 50  0000 C CNN
+	1    8100 3650
+	-1   0    0    -1
+$EndComp
+Wire Wire Line
+	8300 3500 9100 3500
+Wire Wire Line
+	8300 3600 9100 3600
+Wire Wire Line
+	8300 3700 9100 3700
+Wire Wire Line
+	8300 3800 9100 3800
 $EndSCHEMATC

Commit message: KiCad Stepper
Parts:
- added C1, C2, C3: C, symbol C
- added P1: 24V, symbol CONN_01X02
- added P2: CONN_01X02, symbol CONN_01X02
- gave numbers to parts that had none: 5
Connections:
- net +24V: now also C2.1, P1.2 (P2)
- net +5V: now also C1.2, C3.1
- net GND: now also C1.1, C2.2, C3.2, P1.1 (P1)
Other:
- note added: "i2c"
Changed lines of the file:
@@
 LIBS:linear_tech
 LIBS:micrel
+LIBS:microchip_power
 LIBS:NDK
 LIBS:newhaven
@@
 $EndDescr
 $Comp
-L STM32F070CBTx U?
+L STM32F070CBTx U1
 U 1 1 58ADBDAC
 P 3500 3800
-F 0 "U?" H 2500 4650 60  0000 C CNN
+F 0 "U1" H 2500 4650 60  0000 C CNN
 F 1 "STM32F070CBTx" H 3500 3650 60  0000 C CNN
 F 2 "" H 3500 3700 60  0000 C CNN
@@
 $EndComp
 $Comp
-L A4988 U?
+L A4988 U2
 U 1 1 58ADD3F9
 P 5750 3650
-F 0 "U?" H 5500 4150 60  0000 C CNN
+F 0 "U2" H 5500 4150 60  0000 C CNN
 F 1 "A4988" H 5600 3150 60  0000 C CNN
 F 2 "" H 5750 3650 60  0001 C CNN
@@
 $EndComp
 Wire Wire Line
-	4550 3400 5250 3400
-Wire Wire Line
 	4550 3500 5250 3500
 Wire Wire Line
@@
 	4550 4000 5250 4000
 $Comp
-L +5V #PWR?
+L +5V #PWR1
 U 1 1 58ADD77A
-P 5150 3200
-F 0 "#PWR?" H 5150 3050 50  0001 C CNN
-F 1 "+5V" H 5150 3340 50  0000 C CNN
-F 2 "" H 5150 3200 50  0000 C CNN
-F 3 "" H 5150 3200 50  0000 C CNN
-	1    5150 3200
-	1    0    0    -1
-$EndComp
-Wire Wire Line
-	5150 3200 5150 3300
+P 5150 3300
+F 0 "#PWR1" H 5150 3150 50  0001 C CNN
+F 1 "+5V" H 5150 3440 50  0000 C CNN
+F 2 "" H 5150 3300 50  0000 C CNN
+F 3 "" H 5150 3300 50  0000 C CNN
+	1    5150 3300
+	0    -1   -1   0
+$EndComp
 Wire Wire Line
 	5150 3300 5250 3300
 $Comp
-L +24V #PWR?
+L +24V #PWR6
 U 1 1 58ADD82B
-P 6400 3200
-F 0 "#PWR?" H 6400 3050 50  0001 C CNN
-F 1 "+24V" H 6400 3340 50  0000 C CNN
-F 2 "" H 6400 3200 50  0000 C CNN
-F 3 "" H 6400 3200 50  0000 C CNN
-	1    6400 3200
-	1    0    0    -1
-$EndComp
-Wire Wire Line
-	6400 3200 6400 3300
+P 6400 3100
+F 0 "#PWR6" H 6400 2950 50  0001 C CNN
+F 1 "+24V" H 6400 3240 50  0000 C CNN
+F 2 "" H 6400 3100 50  0000 C CNN
+F 3 "" H 6400 3100 50  0000 C CNN
+	1    6400 3100
+	1    0    0    -1
+$EndComp
+Wire Wire Line
+	6400 3100 6400 3300
 Wire Wire Line
 	6400 3300 6250 3300
 $Comp
-L GND #PWR?
+L GND #PWR5
 U 1 1 58ADD8D7
-P 6250 4100
-F 0 "#PWR?" H 6250 3850 50  0001 C CNN
-F 1 "GND" H 6250 3950 50  0000 C CNN
-F 2 "" H 6250 4100 50  0000 C CNN
-F 3 "" H 6250 4100 50  0000 C CNN
-	1    6250 4100
-	1    0    0    -1
-$EndComp
-$Comp
-L +5V #PWR?
-U 1 1 58ADD8EF
-P 6250 3900
-F 0 "#PWR?" H 6250 3750 50  0001 C CNN
-F 1 "+5V" H 6250 4040 50  0000 C CNN
-F 2 "" H 6250 3900 50  0000 C CNN
-F 3 "" H 6250 3900 50  0000 C CNN
-	1    6250 3900
-	0    1    1    0
-$EndComp
-Wire Wire Line
-	6250 4100 6250 4000
-$Comp
-L GND #PWR?
+P 6250 4300
+F 0 "#PWR5" H 6250 4050 50  0001 C CNN
+F 1 "GND" H 6250 4150 50  0000 C CNN
+F 2 "" H 6250 4300 50  0000 C CNN
+F 3 "" H 6250 4300 50  0000 C CNN
+	1    6250 4300
+	1    0    0    -1
+$EndComp
+Wire Wire Line
+	6250 4000 6250 4300
+$Comp
+L GND #PWR8
 U 1 1 58ADD94B
-P 6550 3300
-F 0 "#PWR?" H 6550 3050 50  0001 C CNN
-F 1 "GND" H 6550 3150 50  0000 C CNN
-F 2 "" H 6550 3300 50  0000 C CNN
-F 3 "" H 6550 3300 50  0000 C CNN
-	1    6550 3300
+P 6800 3400
+F 0 "#PWR8" H 6800 3150 50  0001 C CNN
+F 1 "GND" H 6800 3250 50  0000 C CNN
+F 2 "" H 6800 3400 50  0000 C CNN
+F 3 "" H 6800 3400 50  0000 C CNN
+	1    6800 3400
 	-1   0    0    1
 $EndComp
 Wire Wire Line
-	6550 3300 6550 3400
-Wire Wire Line
-	6550 3400 6250 3400
-$Comp
-L Stepper U?
+	6250 3400 6800 3400
+$Comp
+L Stepper U3
 U 1 1 58B01121
 P 9600 3650
-F 0 "U?" H 9350 4000 60  0000 C CNN
+F 0 "U3" H 9350 4000 60  0000 C CNN
 F 1 "Stepper" H 9450 3300 60  0000 C CNN
 F 2 "" H 9600 3650 60  0000 C CNN
@@
 	6250 3800 7100 3800
 $Comp
-L CONN_01X04 P?
+L CONN_01X04 P3
 U 1 1 58D04B64
 P 7300 3650
-F 0 "P?" H 7300 3900 50  0000 C CNN
+F 0 "P3" H 7300 3900 50  0000 C CNN
 F 1 "CONN_01X04" V 7400 3650 50  0000 C CNN
 F 2 "" H 7300 3650 50  0000 C CNN
@@
 $EndComp
 $Comp
-L CONN_01X04 P?
+L CONN_01X04 P4
 U 1 1 58D04BB1
 P 8100 3650
-F 0 "P?" H 8100 3900 50  0000 C CNN
+F 0 "P4" H 8100 3900 50  0000 C CNN
 F 1 "CONN_01X04" V 8200 3650 50  0000 C CNN
 F 2 "" H 8100 3650 50  0000 C CNN
@@
 Wire Wire Line
 	8300 3800 9100 3800
+$Comp
+L CONN_01X02 P1
+U 1 1 58E7C5D7
+P 5300 1350
+F 0 "P1" H 5300 1500 50  0000 C CNN
+F 1 "24V" V 5400 1350 50  0000 C CNN
+F 2 "" H 5300 1350 50  0000 C CNN
+F 3 "" H 5300 1350 50  0000 C CNN
+	1    5300 1350
+	0    -1   -1   0
+$EndComp
+$Comp
+L +24V #PWR4
+U 1 1 58E7C816
+P 5350 1650
+F 0 "#PWR4" H 5350 1500 50  0001 C CNN
+F 1 "+24V" H 5350 1790 50  0000 C CNN
+F 2 "" H 5350 1650 50  0000 C CNN
+F 3 "" H 5350 1650 50  0000 C CNN
+	1    5350 1650
+	-1   0    0    1
+$EndComp
+Wire Wire Line
+	5350 1650 5350 1550
+$Comp
+L GND #PWR3
+U 1 1 58E7C85C
+P 5250 1650
+F 0 "#PWR3" H 5250 1400 50  0001 C CNN
+F 1 "GND" H 5250 1500 50  0000 C CNN
+F 2 "" H 5250 1650 50  0000 C CNN
+F 3 "" H 5250 1650 50  0000 C CNN
+	1    5250 1650
+	1    0    0    -1
+$EndComp
+Wire Wire Line
+	5250 1650 5250 1550
+$Comp
+L C C3
+U 1 1 58E7D29B
+P 6550 4050
+F 0 "C3" H 6575 4150 50  0000 L CNN
+F 1 "C" H 6575 3950 50  0000 L CNN
+F 2 "" H 6588 3900 50  0000 C CNN
+F 3 "" H 6550 4050 50  0000 C CNN
+	1    6550 4050
+	1    0    0    -1
+$EndComp
+Wire Wire Line
+	6250 3900 6750 3900
+Wire Wire Line
+	6250 4200 6550 4200
+Connection ~ 6250 4200
+$Comp
+L +5V #PWR7
+U 1 1 58E7D41C
+P 6750 3900
+F 0 "#PWR7" H 6750 3750 50  0001 C CNN
+F 1 "+5V" H 6750 4040 50  0000 C CNN
+F 2 "" H 6750 3900 50  0000 C CNN
+F 3 "" H 6750 3900 50  0000 C CNN
+	1    6750 3900
+	0    1    1    0
+$EndComp
+Connection ~ 6550 3900
+$Comp
+L C C2
+U 1 1 58E7D597
+P 6550 3250
+F 0 "C2" H 6575 3350 50  0000 L CNN
+F 1 "C" H 6575 3150 50  0000 L CNN
+F 2 "" H 6588 3100 50  0000 C CNN
+F 3 "" H 6550 3250 50  0000 C CNN
+	1    6550 3250
+	1    0    0    -1
+$EndComp
+Wire Wire Line
+	6400 3100 6550 3100
+Connection ~ 6550 3400
+Wire Wire Line
+	4550 3400 5250 3400
+$Comp
+L C C1
+U 1 1 58E7DC37
+P 5200 3150
+F 0 "C1" H 5225 3250 50  0000 L CNN
+F 1 "C" H 5225 3050 50  0000 L CNN
+F 2 "" H 5238 3000 50  0000 C CNN
+F 3 "" H 5200 3150 50  0000 C CNN
+	1    5200 3150
+	1    0    0    -1
+$EndComp
+Connection ~ 5200 3300
+$Comp
+L GND #PWR2
+U 1 1 58E7E12E
+P 5200 3000
+F 0 "#PWR2" H 5200 2750 50  0001 C CNN
+F 1 "GND" H 5200 2850 50  0000 C CNN
+F 2 "" H 5200 3000 50  0000 C CNN
+F 3 "" H 5200 3000 50  0000 C CNN
+	1    5200 3000
+	-1   0    0    1
+$EndComp
+$Comp
+L CONN_01X02 P2
+U 1 1 58E7FD13
+P 5900 6700
+F 0 "P2" H 5900 6850 50  0000 C CNN
+F 1 "CONN_01X02" V 6000 6700 50  0000 C CNN
+F 2 "" H 5900 6700 50  0000 C CNN
+F 3 "" H 5900 6700 50  0000 C CNN
+	1    5900 6700
+	0    1    1    0
+$EndComp
+Wire Notes Line
+	5100 6150 6350 6150
+Wire Notes Line
+	6350 6150 6350 7000
+Wire Notes Line
+	6350 7000 5100 7000
+Wire Notes Line
+	5100 7000 5100 6150
+Text Notes 5150 6100 0    60   ~ 0
+i2c
 $EndSCHEMATC
